File: SensorBrdInterface.sch (KiCad schematic (older format))
At the start: 15 parts, among them J7 MinionConn, J8 CurrentConn, U5 LTC6820, U6 LTC6820, U7 HX1188FNL

Commit message: Adds HX1188 component to common library
Parts:
- U7: symbol utsvt-bps:HX1188FNL -> utsvt-chips:HX1188FNL
Changed lines of the file:
@@
 I_IM
 $Comp
-L utsvt-bps:HX1188FNL U7
+L utsvt-chips:HX1188FNL U7
 U 1 1 5F145AE9
 P 8100 3400
