File: BPS-Leader.kicad_pcb (KiCad board)
At the start: 2 copper layers, 100 x 75 mm, 153 parts, among them J1 GPIO Analyzer, J10 CAN_Out, J11 ErrorLightConn, J12 USB_B_Micro, J13 FanBrdConn, J2 Volt/Temp SPI Analyzer, J3 Current SPI Analyzer, J4 CAN Analyzer, J5 SWD, J6 PowerConn, J7 MinionConn, J8 CurrentConn, J9 ContactorConn, Q1 NTR4003NT1G, Q2 VND5N07-E, Q3 NTR4003NT1G, Q4 VND5N07-E, SW1 B3SL-1002P, U1 STM32F413RHTx, U10 CDSOT23-T24CAN, U11 SI8261ABC-IS, U12 CP2102N-A01-GQFN24, U13 SI8261ABC-IS, U14 SI8261ABC-IS, U15 SI8261ABC-IS, U16 SI8261ABC-IS, U17 MCP112, U18 RN4871-I, U2 RI3-1205S, U3 NCP1117-3.3_SOT223, U4 M24128, U5 LTC6820, U6 LTC6820, U7 HX1188FNL, U8 SI8261ABC-IS, U9 ADM3055E, Y1 8M

Commit message: Updated to KiCAD 6
Other:
- net class Default removed
