File: CAN.kicad_sch (KiCad schematic)
At the start: 17 parts

Commit message: Update repo to only use one common library
Parts:
- gave numbers to parts that had none: 15

Commit message: Fixed all symbol issues
Parts:
- L1: symbol Device:Ferrite_Bead_Small -> Device:FerriteBead_Small
- L2: symbol Device:Ferrite_Bead_Small -> Device:D
Connections:
- net at C29.1, C30.1, C31.1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: now also L1.1
- net at C28.1, U9.19 (V_ISO_Out): now also L1.2
Changed lines of the file:
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@@
     )
   )
-  (symbol (lib_id "Device:Ferrite_Bead_Small") (at 151.13 77.47 270) (unit 1)
+  (symbol (lib_id "Device:FerriteBead_Small") (at 151.13 77.47 270) (unit 1)
     (in_bom yes) (on_board yes) (dnp no)
     (property "Reference" "L1" (at 152.4 74.93 90)
@@
       (effects (font (size 1.27 1.27)) hide)
     )
-    (property "Datasheet" "" (at 151.13 77.47 0)
+    (property "Datasheet" "~" (at 151.13 77.47 0)
       (effects (font (size 1.27 1.27)) hide)
     )
+    (pin "1")
+    (pin "2")
     (instances
       (project "BPS-Leader"
@@
     )
   )
-  (symbol (lib_id "Device:Ferrite_Bead_Small") (at 151.13 85.09 270) (unit 1)
+  (symbol (lib_id "Device:D") (at 151.13 85.09 270) (unit 1)
     (in_bom yes) (on_board yes) (dnp no)
     (property "Reference" "L2" (at 152.4 87.63 90)
@@
       (effects (font (size 1.27 1.27)) hide)
     )
+    (pin "1")
+    (pin "2")
     (instances
       (project "BPS-Leader"
