File: Contactor.kicad_sch (KiCad schematic)
At the start: 20 parts

Commit message: Update repo to only use one common library
Parts:
- gave numbers to parts that had none: 17

Commit message: Fixed all symbol issues
Parts:
- D11: symbol Device:LED_ALT -> Device:D
- D12: symbol Device:D_ALT -> Device:D
Connections:
- net +12V: now also D12.1 (K)
- net CONTACTOR_V-: now also D12.2 (A)
- net at R21.2: now also D11.2 (A)
- net at Q1.3 (D), U8.3 (CATHODE): now also D11.1 (K)
Changed lines of the file:
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@@
     )
   )
-  (symbol (lib_id "Device:D_ALT") (at 139.7 86.36 270) (unit 1)
+  (symbol (lib_id "Device:D") (at 139.7 86.36 270) (unit 1)
     (in_bom yes) (on_board yes) (dnp no)
     (property "Reference" "D12" (at 141.7066 85.1916 90)
@@
       (effects (font (size 1.27 1.27)) hide)
     )
+    (pin "1")
+    (pin "2")
     (instances
       (project "BPS-Leader"
@@
     )
   )
-  (symbol (lib_id "Device:LED_ALT") (at 59.69 93.98 90) (unit 1)
+  (symbol (lib_id "Device:D") (at 59.69 93.98 90) (unit 1)
     (in_bom yes) (on_board yes) (dnp no)
     (property "Reference" "D11" (at 52.07 92.71 90)
@@
       (effects (font (size 1.27 1.27)) hide)
     )
+    (pin "1")
+    (pin "2")
     (instances
       (project "BPS-Leader"
