File: ErrorLight.kicad_sch (KiCad schematic)
At the start: 15 parts

Commit message: Update repo to only use one common library
Parts:
- gave numbers to parts that had none: 15

Commit message: Fixed all symbol issues
Parts:
- D14: symbol Device:LED_ALT -> Device:D
Connections:
- net +5V: now also D14.2 (A)
- net at R30.1: now also D14.1 (K)
Changed lines of the file:
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@@
     )
   )
-  (symbol (lib_id "Device:LED_ALT") (at 102.87 88.9 90) (unit 1)
+  (symbol (lib_id "Device:D") (at 102.87 88.9 90) (unit 1)
     (in_bom yes) (on_board yes) (dnp no)
     (property "Reference" "D14" (at 105.8418 87.9348 90)
@@
       (effects (font (size 1.27 1.27)) hide)
     )
+    (property "Sim.Device" "D" (at 102.87 88.9 0)
+      (effects (font (size 1.27 1.27)) hide)
+    )
+    (property "Sim.Pins" "1=K 2=A" (at 102.87 88.9 0)
+      (effects (font (size 1.27 1.27)) hide)
+    )
+    (pin "1")
+    (pin "2")
     (instances
       (project "BPS-Leader"
