File: LEDs.kicad_sch (KiCad schematic)
At the start: 18 parts

Commit message: Update repo to only use one common library
Parts:
- gave numbers to parts that had none: 9

Commit message: Fixed all symbol issues
Parts:
- D10, D2, D3, D4, D5, D6, D7, D8, D9: symbol Device:LED_ALT -> Device:D
Connections:
- net PA4: now also D5.2 (A)
- net PA5: now also D4.2 (A)
- net PA6: now also D3.2 (A)
- net PA7: now also D2.2 (A)
- net PC0: now also D10.2 (A)
- net PC1: now also D9.2 (A)
- net PC2: now also D8.2 (A)
- net PC3: now also D7.2 (A)
- net PC4: now also D6.2 (A)
- net at R8.1: now also D6.1 (K)
- net at R4.1: now also D2.1 (K)
- net at R5.1: now also D3.1 (K)
- net at R6.1: now also D4.1 (K)
- net at R7.1: now also D5.1 (K)
- net at R9.1: now also D7.1 (K)
- net at R11.1: now also D9.1 (K)
- net at R10.1: now also D8.1 (K)
- net at R12.1: now also D10.1 (K)
Changed lines of the file:
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@@
     (effects (font (size 1.27 1.27)) (justify left))
   )
-  (symbol (lib_id "Device:LED_ALT") (at 147.32 78.74 90) (unit 1)
+  (symbol (lib_id "Device:D") (at 147.32 78.74 90) (unit 1)
     (in_bom yes) (on_board yes) (dnp no)
     (property "Reference" "D6" (at 150.2918 77.7748 90)
@@
       (effects (font (size 1.27 1.27)) hide)
     )
+    (pin "1")
+    (pin "2")
     (instances
       (project "BPS-Leader"
@@
     )
   )
-  (symbol (lib_id "Device:LED_ALT") (at 93.98 78.74 90) (unit 1)
+  (symbol (lib_id "Device:D") (at 93.98 78.74 90) (unit 1)
     (in_bom yes) (on_board yes) (dnp no)
     (property "Reference" "D2" (at 96.9772 77.7748 90)
@@
       (effects (font (size 1.27 1.27)) hide)
     )
+    (pin "1")
+    (pin "2")
     (instances
       (project "BPS-Leader"
@@
     )
   )
-  (symbol (lib_id "Device:LED_ALT") (at 104.14 78.74 90) (unit 1)
+  (symbol (lib_id "Device:D") (at 104.14 78.74 90) (unit 1)
     (in_bom yes) (on_board yes) (dnp no)
     (property "Reference" "D3" (at 107.1372 77.7748 90)
@@
       (effects (font (size 1.27 1.27)) hide)
     )
+    (pin "1")
+    (pin "2")
     (instances
       (project "BPS-Leader"
@@
     )
   )
-  (symbol (lib_id "Device:LED_ALT") (at 114.3 78.74 90) (unit 1)
+  (symbol (lib_id "Device:D") (at 114.3 78.74 90) (unit 1)
     (in_bom yes) (on_board yes) (dnp no)
     (property "Reference" "D4" (at 117.2972 77.7748 90)
@@
       (effects (font (size 1.27 1.27)) hide)
     )
+    (pin "1")
+    (pin "2")
     (instances
       (project "BPS-Leader"
@@
     )
   )
-  (symbol (lib_id "Device:LED_ALT") (at 124.46 78.74 90) (unit 1)
+  (symbol (lib_id "Device:D") (at 124.46 78.74 90) (unit 1)
     (in_bom yes) (on_board yes) (dnp no)
     (property "Reference" "D5" (at 127.4318 77.7748 90)
@@
       (effects (font (size 1.27 1.27)) hide)
     )
+    (pin "1")
+    (pin "2")
     (instances
       (project "BPS-Leader"
@@
     )
   )
-  (symbol (lib_id "Device:LED_ALT") (at 167.64 78.74 90) (unit 1)
+  (symbol (lib_id "Device:D") (at 167.64 78.74 90) (unit 1)
     (in_bom yes) (on_board yes) (dnp no)
     (property "Reference" "D7" (at 170.6118 77.7748 90)
@@
       (effects (font (size 1.27 1.27)) hide)
     )
+    (pin "1")
+    (pin "2")
     (instances
       (project "BPS-Leader"
@@
     )
   )
-  (symbol (lib_id "Device:LED_ALT") (at 193.04 78.74 90) (unit 1)
+  (symbol (lib_id "Device:D") (at 193.04 78.74 90) (unit 1)
     (in_bom yes) (on_board yes) (dnp no)
     (property "Reference" "D9" (at 196.0118 77.7748 90)
@@
       (effects (font (size 1.27 1.27)) hide)
     )
+    (pin "1")
+    (pin "2")
     (instances
       (project "BPS-Leader"
@@
     )
   )
-  (symbol (lib_id "Device:LED_ALT") (at 180.34 78.74 90) (unit 1)
+  (symbol (lib_id "Device:D") (at 180.34 78.74 90) (unit 1)
     (in_bom yes) (on_board yes) (dnp no)
     (property "Reference" "D8" (at 183.3118 77.7748 90)
@@
       (effects (font (size 1.27 1.27)) hide)
     )
+    (pin "1")
+    (pin "2")
     (instances
       (project "BPS-Leader"
@@
     )
   )
-  (symbol (lib_id "Device:LED_ALT") (at 205.74 78.74 90) (unit 1)
+  (symbol (lib_id "Device:D") (at 205.74 78.74 90) (unit 1)
     (in_bom yes) (on_board yes) (dnp no)
     (property "Reference" "D10" (at 208.7118 77.7748 90)
@@
       (effects (font (size 1.27 1.27)) hide)
     )
-    (instances
-      (project "BPS-Leader"
+    (pin "1")
+    (pin "2")
+    (instances
+      (project "BPS-Leader"
