File: PowerDist.kicad_sch (KiCad schematic)
At the start: 13 parts

Commit message: Update repo to only use one common library
Parts:
- gave numbers to parts that had none: 12

Commit message: Fixed all symbol issues
Parts:
- D1: symbol Device:LED_ALT -> Device:D
Connections:
- net GND: now also D1.1 (K)
- net at R1.2: now also D1.2 (A)
Changed lines of the file:
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@@
     )
   )
-  (symbol (lib_id "Device:LED_ALT") (at 161.29 91.44 90) (unit 1)
+  (symbol (lib_id "Device:D") (at 161.29 91.44 90) (unit 1)
     (in_bom yes) (on_board yes) (dnp no)
     (property "Reference" "D1" (at 164.2872 90.4748 90)
@@
       (effects (font (size 1.27 1.27)) hide)
     )
+    (property "Sim.Device" "D" (at 161.29 91.44 0)
+      (effects (font (size 1.27 1.27)) hide)
+    )
+    (property "Sim.Pins" "1=K 2=A" (at 161.29 91.44 0)
+      (effects (font (size 1.27 1.27)) hide)
+    )
+    (pin "1")
+    (pin "2")
     (instances
       (project "BPS-Leader"
