File: USB.kicad_sch (KiCad schematic)
At the start: 8 parts, among them U12 CP2102N-A01-GQFN24

Commit message: Update repo to only use one common library
Parts:
- gave numbers to parts that had none: 7

Commit message: Fixed all symbol issues
Parts:
- U12: symbol Interface_USB:CP2102N-A01-GQFN24 -> Interface_USB:CP2102N-Axx-xQFN24
Connections:
- net +3.3V: now also U12.5 (VIO), U12.6 (VDD), U12.7 (VREGIN)
- net GND: now also U12.2 (GND), U12.25 (GND)
- net UART_RX: now also U12.21 (TXD)
- net UART_TX: now also U12.20 (RXD)
- net at D15.3 (K), J12.2 (D-): now also U12.4 (D-)
- net at D15.4 (K), J12.3 (D+): now also U12.3 (D+)
- net at R34.1, R35.1: now also U12.8 (VBUS)
- net at R36.2: now also U12.9 (~{RST})
Other:
- moved on the sheet: C35, C36, D15, J12, R34, R35, R36
